File: carte/interfaceI2C_eCAN/dsPIC_I2C.sch (EAGLE design)
At the start: 54 parts, among them IC2 DSPIC33FJ128MC804PT, J1 RJ11-2L-B, J9 22-27-2051, Q2 BSS123, Q4 BSS123, U2 LP2985-33DBVR

Commit message: update dsPIC_I2C
Petite mise en forme des sch et brd
rajout d'un README
Other:
- moved on the sheet: C1, C11, C12, C13, C14, C15, C2, C3, C4, C6, FERRITE1, FERRITE2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
