File: carte/alimentation/alimentation.brd (EAGLE design)
At the start: 160 x 100 mm, 26 parts, among them IC1 LM2596T, K1 RP811005, T1 2N2222, X10 22-23-2021, X11 22-23-2021, X9 22-23-2021

Commit message: MAJ ancienne carte alim
Connections:
- removed net N$2: D4.C, K1.11, K1.A1, R1.1, R4.1, X15.2
- new net BOBINE: D4.A, K1.A2, R3.2, R7.2
- net BOB: now also D4.C, K1.11, K1.A1, R1.1, R4.1, X15.2; no longer D4.A, K1.A2, R3.2, R7.2
Changed lines of the file:
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@@
 <?xml version="1.0" encoding="utf-8"?>
 <!DOCTYPE eagle SYSTEM "eagle.dtd">
-<eagle version="8.1.0">
+<eagle version="9.0.0">
 <drawing>
 <settings>
 <setting alwaysvectorfont="no"/>
+<setting keepoldvectorfont="yes"/>
 <setting verticaltext="up"/>
 </settings>
@@
 <param name="dpMaxLengthDifference" value="10mm"/>
 <param name="dpGapFactor" value="2.5"/>
-<param name="checkGrid" value="0"/>
 <param name="checkAngle" value="0"/>
 <param name="checkFont" value="1"/>
 <param name="checkRestrict" value="1"/>
+<param name="checkStop" value="0"/>
+<param name="checkValues" value="0"/>
 <param name="useDiameter" value="13"/>
 <param name="maxErrors" value="50"/>
@@
 </signal>
 <signal name="BOB">
-<contactref element="K1" pad="A2"/>
-<contactref element="R3" pad="2"/>
-<contactref element="R7" pad="2"/>
-<contactref element="D4" pad="A"/>
-<wire x1="-60.01" y1="-10.16" x2="-60.01" y2="-102.87" width="0" layer="19" extent="1-1"/>
-<wire x1="-40.54" y1="55.85" x2="-60.01" y2="-10.16" width="0" layer="19" extent="1-1"/>
-<wire x1="-44.45" y1="-240.03" x2="-60.01" y2="-102.87" width="0" layer="19" extent="1-1"/>
-</signal>
-<signal name="N$2">
 <contactref element="R4" pad="1"/>
-<contactref element="D4" pad="C"/>
 <contactref element="X15" pad="2"/>
 <contactref element="K1" pad="11"/>
+<contactref element="R1" pad="1"/>
 <contactref element="K1" pad="A1"/>
-<contactref element="R1" pad="1"/>
+<contactref element="D4" pad="C"/>
 <wire x1="-49.57" y1="-173.99" x2="-61.91" y2="-186.69" width="0" layer="19" extent="1-1"/>
 <wire x1="-54.61" y1="-240.03" x2="-61.91" y2="-186.69" width="0" layer="19" extent="1-1"/>
@@
 <wire x1="-32.68" y1="62.36" x2="-60.01" y2="-83.82" width="0" layer="19" extent="1-1"/>
 </signal>
+<signal name="BOBINE">
+<contactref element="D4" pad="A"/>
+<contactref element="K1" pad="A2"/>
+<contactref element="R3" pad="2"/>
+<contactref element="R7" pad="2"/>
+<wire x1="-60.01" y1="-10.16" x2="-60.01" y2="-102.87" width="0" layer="19" extent="1-1"/>
+<wire x1="-40.54" y1="55.85" x2="-60.01" y2="-10.16" width="0" layer="19" extent="1-1"/>
+<wire x1="-44.45" y1="-240.03" x2="-60.01" y2="-102.87" width="0" layer="19" extent="1-1"/>
+</signal>
 </signals>
