File: carte/alimentation/update_alimentation.sch (EAGLE design)
At the start: 95 parts, among them IC1 LM2596T, IC2 LM2596T, IC4 DSPIC33FJ128MC804PT, J4 RJ11-2L-B, U2 LP2985-33DBVR, X10 22-23-2021, X11 22-23-2021, X9 22-23-2021

Commit message: MAJ carte alim sch/brd
Parts:
- added R10, R11: 560, resistor:R-EU_R0805
- added R12: 300, resistor:R-EU_R0805
- added R13: 820, resistor:R-EU_R0805
- added R14: 240, resistor:R-EU_R0805
- added R15, R16: 200, resistor:R-EU_R0805
- added R17: 1600, resistor:R-EU_R0805
- added R18: 1100, resistor:R-EU_R0805
- added R19: 220, resistor:R-EU_R0805
- added R20: 1300, resistor:R-EU_R0805
- added R9: 270, resistor:R-EU_R0805
Connections:
- net N$6 renamed BAT3+
- removed net N$3: X13-2.KL, X14-1.KL
- removed net N$4: X14-2.KL, X15-1.KL
- new net BAT12_11.1V: J2.4, J3.1, R13.1, X14-2.KL, X15-1.KL
- new net BAT1_3.7V: J3.3, R9.1
- new net BAT1_7.4V: J3.2, R11.1
- new net BAT23_22.2V: J1.4, J2.1, R17.1, X13-2.KL, X14-1.KL
- new net BAT2_14.8V: J2.3, R18.1
- new net BAT2_18.5V: J2.2, R20.1
- new net BAT3_25.9V: J1.3
- new net BAT3_29.6V: J1.2
- new net BAT3_33.3V: J1.1
- new net N$20: R10.2, R9.2
- new net N$21: R11.2, R12.2
- new net N$22: R13.2, R14.2
- new net N$23: R18.2, R19.2
- new net N$24: R15.2, R20.2
- new net N$25: R16.2, R17.2
- net GND: now also R10.1, R12.1, R14.1, R15.1, R16.1, R19.1; no longer J1.4, J2.4
Other:
- moved on the sheet: J1, J2, J3

Commit message: MaJ carte alim : modification labels
Connections:
- net +5V: no longer C6.2, D5.C, PC2.+, SL1.2, U$6G$1.1, U2.IN, U2.ON/!OFF
- net +5V_3A: now also C6.2, D5.C, PC2.+, SL1.2, U$6G$1.1, U2.IN, U2.ON/!OFF
Changed lines of the file:
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@@
 <setting verticaltext="up"/>
 </settings>
-<grid distance="0.01" unitdist="inch" unit="inch" style="lines" multiple="1" display="no" altdistance="0.01" altunitdist="inch" altunit="inch"/>
+<grid distance="0.1" unitdist="inch" unit="inch" style="lines" multiple="1" display="no" altdistance="0.01" altunitdist="inch" altunit="inch"/>
 <layers>
 <layer number="1" name="Top" color="4" fill="1" visible="no" active="no"/>
@@
 <wire x1="93.977509375" y1="153.043534375" x2="93.98" y2="153.043534375" width="0.1524" layer="91"/>
 </segment>
-</net>
-<net name="N$9" class="0">
-<segment>
-<pinref part="IC2" gate="G$1" pin="OUT"/>
-<pinref part="U$5" gate="G$1" pin="C"/>
-<wire x1="60.96" y1="-12.7" x2="63.5" y2="-12.7" width="0.1524" layer="91"/>
-<wire x1="63.5" y1="-12.7" x2="63.5" y2="-7.62" width="0.1524" layer="91"/>
-<pinref part="U$11" gate="G$1" pin="1"/>
-<wire x1="63.5" y1="-12.7" x2="68.326" y2="-12.7" width="0.1524" layer="91"/>
-<junction x="63.5" y="-12.7"/>
-</segment>
-</net>
-<net name="+5V" class="0">
-<segment>
-<pinref part="P+1" gate="1" pin="+5V"/>
-<wire x1="88.897509375" y1="-4.436465625" x2="88.9" y2="-4.436465625" width="0.1524" layer="91"/>
-<wire x1="88.9" y1="-4.436465625" x2="88.9" y2="-12.7" width="0.1524" layer="91"/>
-<pinref part="IC2" gate="G$1" pin="FB"/>
-<wire x1="88.9" y1="-12.7" x2="88.9" y2="-17.78" width="0.1524" layer="91"/>
-<wire x1="60.96" y1="-17.78" x2="88.9" y2="-17.78" width="0.1524" layer="91"/>
-<pinref part="C1" gate="G$1" pin="+"/>
-<wire x1="88.9" y1="-17.78" x2="88.9" y2="-20.32" width="0.1524" layer="91"/>
-<junction x="88.9" y="-17.78"/>
-<pinref part="U$11" gate="G$1" pin="2"/>
-<wire x1="83.566" y1="-12.7" x2="88.9" y2="-12.7" width="0.1524" layer="91"/>
-<junction x="88.9" y="-12.7"/>
-</segment>
-<segment>
-<wire x1="467.36" y1="198.12" x2="467.36" y2="205.74" width="0.1524" layer="91"/>
-<pinref part="P+5" gate="1" pin="+5V"/>
-<wire x1="467.36" y1="205.74" x2="457.2" y2="205.74" width="0.1524" layer="91"/>
-<wire x1="457.2" y1="205.74" x2="457.2" y2="198.12" width="0.1524" layer="91"/>
-<junction x="467.36" y="205.74"/>
-<pinref part="R1" gate="G$1" pin="2"/>
-<pinref part="R6" gate="G$1" pin="2"/>
-</segment>
-<segment>
-<wire x1="482.6" y1="200.66" x2="482.6" y2="198.12" width="0.1524" layer="91"/>
-<wire x1="482.6" y1="198.12" x2="482.6" y2="193.04" width="0.1524" layer="91"/>
-<wire x1="477.52" y1="198.12" x2="482.6" y2="198.12" width="0.1524" layer="91"/>
-<junction x="482.6" y="198.12"/>
-<pinref part="P+9" gate="1" pin="+5V"/>
-<pinref part="C8" gate="G$1" pin="2"/>
+<segment>
+<wire x1="518.16" y1="198.12" x2="520.7" y2="198.12" width="0.1524" layer="91"/>
+<wire x1="520.7" y1="193.04" x2="518.16" y2="193.04" width="0.1524" layer="91"/>
+<wire x1="518.16" y1="193.04" x2="518.16" y2="198.12" width="0.1524" layer="91"/>
+<wire x1="518.16" y1="198.12" x2="518.16" y2="200.66" width="0.1524" layer="91"/>
+<wire x1="510.54" y1="198.12" x2="518.16" y2="198.12" width="0.1524" layer="91"/>
+<junction x="518.16" y="198.12"/>
+<junction x="518.16" y="198.12"/>
+<label x="510.54" y="198.12" size="1.778" layer="95"/>
+<pinref part="P+10" gate="1" pin="+5V"/>
+<pinref part="U2" gate="G$1" pin="IN"/>
+<pinref part="U2" gate="G$1" pin="ON/!OFF"/>
 </segment>
 <segment>
@@
 </segment>
 <segment>
-<wire x1="518.16" y1="198.12" x2="520.7" y2="198.12" width="0.1524" layer="91"/>
-<wire x1="520.7" y1="193.04" x2="518.16" y2="193.04" width="0.1524" layer="91"/>
-<wire x1="518.16" y1="193.04" x2="518.16" y2="198.12" width="0.1524" layer="91"/>
-<wire x1="518.16" y1="198.12" x2="518.16" y2="200.66" width="0.1524" layer="91"/>
-<wire x1="510.54" y1="198.12" x2="518.16" y2="198.12" width="0.1524" layer="91"/>
-<junction x="518.16" y="198.12"/>
-<junction x="518.16" y="198.12"/>
-<label x="510.54" y="198.12" size="1.778" layer="95"/>
-<pinref part="P+10" gate="1" pin="+5V"/>
-<pinref part="U2" gate="G$1" pin="IN"/>
-<pinref part="U2" gate="G$1" pin="ON/!OFF"/>
+<pinref part="U$6" gate="G$1" pin="1"/>
+<wire x1="25.4" y1="83.82" x2="25.4" y2="93.98" width="0.1524" layer="91"/>
+<wire x1="25.4" y1="93.98" x2="35.56" y2="93.98" width="0.1524" layer="91"/>
+<pinref part="D5" gate="1" pin="C"/>
+<wire x1="35.56" y1="93.98" x2="45.72" y2="93.98" width="0.1524" layer="91"/>
+<wire x1="45.72" y1="93.98" x2="45.72" y2="81.28" width="0.1524" layer="91"/>
+<wire x1="35.56" y1="93.98" x2="35.56" y2="99.06" width="0.1524" layer="91"/>
+<junction x="35.56" y="93.98"/>
+<label x="35.56" y="99.06" size="1.778" layer="95" xref="yes"/>
+</segment>
+</net>
+<net name="N$9" class="0">
+<segment>
+<pinref part="IC2" gate="G$1" pin="OUT"/>
+<pinref part="U$5" gate="G$1" pin="C"/>
+<wire x1="60.96" y1="-12.7" x2="63.5" y2="-12.7" width="0.1524" layer="91"/>
+<wire x1="63.5" y1="-12.7" x2="63.5" y2="-7.62" width="0.1524" layer="91"/>
+<pinref part="U$11" gate="G$1" pin="1"/>
+<wire x1="63.5" y1="-12.7" x2="68.326" y2="-12.7" width="0.1524" layer="91"/>
+<junction x="63.5" y="-12.7"/>
+</segment>
+</net>
+<net name="+5V" class="0">
+<segment>
+<pinref part="P+1" gate="1" pin="+5V"/>
+<wire x1="88.897509375" y1="-4.436465625" x2="88.9" y2="-4.436465625" width="0.1524" layer="91"/>
+<wire x1="88.9" y1="-4.436465625" x2="88.9" y2="-12.7" width="0.1524" layer="91"/>
+<pinref part="IC2" gate="G$1" pin="FB"/>
+<wire x1="88.9" y1="-12.7" x2="88.9" y2="-17.78" width="0.1524" layer="91"/>
+<wire x1="60.96" y1="-17.78" x2="88.9" y2="-17.78" width="0.1524" layer="91"/>
+<pinref part="C1" gate="G$1" pin="+"/>
+<wire x1="88.9" y1="-17.78" x2="88.9" y2="-20.32" width="0.1524" layer="91"/>
+<junction x="88.9" y="-17.78"/>
+<pinref part="U$11" gate="G$1" pin="2"/>
+<wire x1="83.566" y1="-12.7" x2="88.9" y2="-12.7" width="0.1524" layer="91"/>
+<junction x="88.9" y="-12.7"/>
+</segment>
+<segment>
+<wire x1="467.36" y1="198.12" x2="467.36" y2="205.74" width="0.1524" layer="91"/>
+<pinref part="P+5" gate="1" pin="+5V"/>
+<wire x1="467.36" y1="205.74" x2="457.2" y2="205.74" width="0.1524" layer="91"/>
+<wire x1="457.2" y1="205.74" x2="457.2" y2="198.12" width="0.1524" layer="91"/>
+<junction x="467.36" y="205.74"/>
+<pinref part="R1" gate="G$1" pin="2"/>
+<pinref part="R6" gate="G$1" pin="2"/>
+</segment>
+<segment>
+<wire x1="482.6" y1="200.66" x2="482.6" y2="198.12" width="0.1524" layer="91"/>
+<wire x1="482.6" y1="198.12" x2="482.6" y2="193.04" width="0.1524" layer="91"/>
+<wire x1="477.52" y1="198.12" x2="482.6" y2="198.12" width="0.1524" layer="91"/>
+<junction x="482.6" y="198.12"/>
+<pinref part="P+9" gate="1" pin="+5V"/>
+<pinref part="C8" gate="G$1" pin="2"/>
 </segment>
 <segment>
@@
 <label x="571.5" y="-48.26" size="1.778" layer="95"/>
 </segment>
-<segment>
-<pinref part="U$6" gate="G$1" pin="1"/>
-<wire x1="25.4" y1="83.82" x2="25.4" y2="93.98" width="0.1524" layer="91"/>
-<wire x1="25.4" y1="93.98" x2="35.56" y2="93.98" width="0.1524" layer="91"/>
-<pinref part="D5" gate="1" pin="C"/>
-<wire x1="35.56" y1="93.98" x2="45.72" y2="93.98" width="0.1524" layer="91"/>
-<wire x1="45.72" y1="93.98" x2="45.72" y2="81.28" width="0.1524" layer="91"/>
-<wire x1="35.56" y1="93.98" x2="35.56" y2="99.06" width="0.1524" layer="91"/>
-<junction x="35.56" y="93.98"/>
-<label x="35.56" y="99.06" size="1.778" layer="95" xref="yes"/>
-</segment>
 </net>

Commit message: Modif board + ajout excel
Connections:
- removed net N$20: R10.2, R9.2
- removed net N$21: R11.2, R12.2
- removed net N$22: R13.2, R14.2
- removed net N$23: R18.2, R19.2
- removed net N$24: R15.2, R20.2
- removed net N$25: R16.2, R17.2
- net AN0/RA0: now also R10.2, R9.2
- net AN1/RA1: now also R11.2, R12.2
- net RP16/RC0/AN6: now also R15.2, R20.2
- net RP17/RC1/AN7: now also R16.2, R17.2
- net RP2/RB2/AN4: now also R13.2, R14.2
- net RP3/RB3/AN5: now also R18.2, R19.2
Changed lines of the file:
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@@
 <label x="645.16" y="12.7" size="1.778" layer="95"/>
+</segment>
+<segment>
+<pinref part="R17" gate="G$1" pin="2"/>
+<pinref part="R16" gate="G$1" pin="2"/>
+<wire x1="261.874" y1="73.406" x2="269.494" y2="73.406" width="0.1524" layer="91"/>
+<wire x1="269.494" y1="73.406" x2="269.494" y2="68.326" width="0.1524" layer="91"/>
+<wire x1="269.494" y1="73.406" x2="292.608" y2="73.406" width="0.1524" layer="91"/>
+<junction x="269.494" y="73.406"/>
+<label x="284.48" y="73.66" size="1.778" layer="95"/>
 </segment>
 </net>
@@
 <wire x1="640.08" y1="10.16" x2="665.48" y2="10.16" width="0.1524" layer="91"/>
 <label x="645.16" y="10.16" size="1.778" layer="95"/>
+</segment>
+<segment>
+<pinref part="R20" gate="G$1" pin="2"/>
+<pinref part="R15" gate="G$1" pin="2"/>
+<wire x1="261.874" y1="98.806" x2="269.494" y2="98.806" width="0.1524" layer="91"/>
+<wire x1="269.494" y1="98.806" x2="269.494" y2="93.726" width="0.1524" layer="91"/>
+<wire x1="269.494" y1="98.806" x2="292.862" y2="98.806" width="0.1524" layer="91"/>
+<junction x="269.494" y="98.806"/>
+<label x="284.48" y="99.06" size="1.778" layer="95"/>
 </segment>
 </net>
@@
 <pinref part="PAD4" gate="1" pin="P"/>
 </segment>
+<segment>
+<pinref part="R18" gate="G$1" pin="2"/>
+<pinref part="R19" gate="G$1" pin="2"/>
+<wire x1="261.874" y1="124.206" x2="269.494" y2="124.206" width="0.1524" layer="91"/>
+<wire x1="269.494" y1="124.206" x2="269.494" y2="119.126" width="0.1524" layer="91"/>
+<wire x1="269.494" y1="124.206" x2="292.862" y2="124.206" width="0.1524" layer="91"/>
+<junction x="269.494" y="124.206"/>
+<label x="281.94" y="124.46" size="1.778" layer="95"/>
+</segment>
 </net>
 <net name="RP2/RB2/AN4" class="0">
@@
 <pinref part="PAD3" gate="1" pin="P"/>
 </segment>
+<segment>
+<pinref part="R13" gate="G$1" pin="2"/>
+<pinref part="R14" gate="G$1" pin="2"/>
+<wire x1="261.874" y1="147.066" x2="269.494" y2="147.066" width="0.1524" layer="91"/>
+<wire x1="269.494" y1="147.066" x2="269.494" y2="141.986" width="0.1524" layer="91"/>
+<wire x1="269.494" y1="147.066" x2="293.116" y2="147.066" width="0.1524" layer="91"/>
+<label x="281.94" y="147.32" size="1.778" layer="95"/>
+</segment>
 </net>
 <net name="PWM1L2/RP13/RB13" class="0">
@@
 <pinref part="IC4" gate="G$1" pin="AN0/VREF+/CN2/RA0"/>
 <pinref part="PAD1" gate="1" pin="P"/>
+</segment>
+<segment>
+<pinref part="R9" gate="G$1" pin="2"/>
+<pinref part="R10" gate="G$1" pin="2"/>
+<wire x1="261.874" y1="195.326" x2="269.494" y2="195.326" width="0.1524" layer="91"/>
+<wire x1="269.494" y1="195.326" x2="269.494" y2="190.246" width="0.1524" layer="91"/>
+<wire x1="269.494" y1="195.326" x2="292.1" y2="195.326" width="0.1524" layer="91"/>
+<junction x="269.494" y="195.326"/>
+<label x="281.94" y="195.58" size="1.778" layer="95"/>
 </segment>
 </net>
@@
 <pinref part="IC4" gate="G$1" pin="AN1/VREF-/CN3/RA1"/>
 <pinref part="PAD2" gate="1" pin="P"/>
+</segment>
+<segment>
+<pinref part="R11" gate="G$1" pin="2"/>
+<pinref part="R12" gate="G$1" pin="2"/>
+<wire x1="261.874" y1="169.926" x2="269.494" y2="169.926" width="0.1524" layer="91"/>
+<wire x1="269.494" y1="169.926" x2="269.494" y2="164.846" width="0.1524" layer="91"/>
+<wire x1="269.494" y1="169.926" x2="293.37" y2="169.926" width="0.1524" layer="91"/>
+<junction x="269.494" y="169.926"/>
+<label x="281.94" y="170.18" size="1.778" layer="95"/>
 </segment>
 </net>
@@
 </segment>
 </net>
-<net name="N$20" class="0">
-<segment>
-<pinref part="R9" gate="G$1" pin="2"/>
-<pinref part="R10" gate="G$1" pin="2"/>
-<wire x1="261.874" y1="195.326" x2="269.494" y2="195.326" width="0.1524" layer="91"/>
-<wire x1="269.494" y1="195.326" x2="269.494" y2="190.246" width="0.1524" layer="91"/>
-<wire x1="269.494" y1="195.326" x2="292.1" y2="195.326" width="0.1524" layer="91"/>
-<junction x="269.494" y="195.326"/>
-</segment>
-</net>
-<net name="N$21" class="0">
-<segment>
-<pinref part="R11" gate="G$1" pin="2"/>
-<pinref part="R12" gate="G$1" pin="2"/>
-<wire x1="261.874" y1="169.926" x2="269.494" y2="169.926" width="0.1524" layer="91"/>
-<wire x1="269.494" y1="169.926" x2="269.494" y2="164.846" width="0.1524" layer="91"/>
-<wire x1="269.494" y1="169.926" x2="293.37" y2="169.926" width="0.1524" layer="91"/>
-<junction x="269.494" y="169.926"/>
-</segment>
-</net>
-<net name="N$22" class="0">
-<segment>
-<pinref part="R13" gate="G$1" pin="2"/>
-<pinref part="R14" gate="G$1" pin="2"/>
-<wire x1="261.874" y1="147.066" x2="269.494" y2="147.066" width="0.1524" layer="91"/>
-<wire x1="269.494" y1="147.066" x2="269.494" y2="141.986" width="0.1524" layer="91"/>
-<wire x1="269.494" y1="147.066" x2="293.116" y2="147.066" width="0.1524" layer="91"/>
-</segment>
-</net>
-<net name="N$23" class="0">
-<segment>
-<pinref part="R18" gate="G$1" pin="2"/>
-<pinref part="R19" gate="G$1" pin="2"/>
-<wire x1="261.874" y1="124.206" x2="269.494" y2="124.206" width="0.1524" layer="91"/>
-<wire x1="269.494" y1="124.206" x2="269.494" y2="119.126" width="0.1524" layer="91"/>
-<wire x1="269.494" y1="124.206" x2="292.862" y2="124.206" width="0.1524" layer="91"/>
-<junction x="269.494" y="124.206"/>
-</segment>
-</net>
-<net name="N$24" class="0">
-<segment>
-<pinref part="R20" gate="G$1" pin="2"/>
-<pinref part="R15" gate="G$1" pin="2"/>
-<wire x1="261.874" y1="98.806" x2="269.494" y2="98.806" width="0.1524" layer="91"/>
-<wire x1="269.494" y1="98.806" x2="269.494" y2="93.726" width="0.1524" layer="91"/>
-<wire x1="269.494" y1="98.806" x2="292.862" y2="98.806" width="0.1524" layer="91"/>
-<junction x="269.494" y="98.806"/>
-</segment>
-</net>
-<net name="N$25" class="0">
-<segment>
-<pinref part="R17" gate="G$1" pin="2"/>
-<pinref part="R16" gate="G$1" pin="2"/>
-<wire x1="261.874" y1="73.406" x2="269.494" y2="73.406" width="0.1524" layer="91"/>
-<wire x1="269.494" y1="73.406" x2="269.494" y2="68.326" width="0.1524" layer="91"/>
-<wire x1="269.494" y1="73.406" x2="292.608" y2="73.406" width="0.1524" layer="91"/>
-<junction x="269.494" y="73.406"/>
-</segment>
-</net>
