File: carte/alimentation/Alimv1.brd (EAGLE design)
At the start: 160 x 100 mm, 95 parts, among them IC1 LM2596T, IC2 LM2596T, IC4 DSPIC33FJ128MC804PT, J4 RJ11-2L-B, U2 LP2985-33DBVR, X10 22-23-2021, X11 22-23-2021, X9 22-23-2021

Commit message: alim v1
Reprise du travail des élèves
Parts:
- removed C8: 100n, SmartPrj:C0603-ROUND
- removed C9: 100n, SmartPrj:C0603K
- removed J1: (no value), con-amp:10X04MTA
- removed PAD1: (no value), wirepad:1,6/0,9
- removed PC2: 47u, rcl:PANASONIC_D
- removed SL1: (no value), con-amp-quick:02P
- removed X12: (no value), con-wago-500:W237-102
- added R10, R11, R12, R13, R14, R9: 20k, LibPerso:R0805
- added R15: 0, LibPerso:R0805
- added U$13: NX3L4051PW, Robot_MT:SOT403
- added X2, X3: MSTBV2, con-phoenix-508:MSTBV2
- added X4: 1751248, con-phoenix-350:1751248
- X1: value (none) -> MSTBV2; device con-wago-500:W237-102 -> con-phoenix-508:MSTBV2
- moved SL2 162.3 mm to (157.5, 31.8)
- moved C4 118.3 mm to (115.6, 81.3), turned to 180 degrees
- moved C26 103.3 mm to (87.6, 81.3), turned to 180 degrees
- moved U$11 90.0 mm to (120.7, 66.0)
- moved U$7 88.7 mm to (35.6, 52.1), turned to 180 degrees
- moved PAD2 88.0 mm to (134.6, 5.08)
- moved D5 85.0 mm to (25.4, 52.1)
- moved PAD5 81.4 mm to (134.6, 7.62)
- moved C29 80.4 mm to (73.7, 81.3), turned to 0 degrees
- moved PAD6 78.8 mm to (134.6, 10.2)
- moved U$5 78.7 mm to (110.5, 67.3), turned to 270 degrees
- moved U$3 78.3 mm to (68.6, 45.7)
- moved PAD3 76.0 mm to (134.6, 12.7)
- moved C14 74.5 mm to (101.5, 4.06), turned to 180 degrees
- moved RESET 74.5 mm to (116.2, 5.08), turned to 180 degrees
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Connections:
- net N$3 renamed BAT23_22.2V
- net N$4 renamed BAT12_11.1V
- net N$6 renamed BAT3+
- removed net +5V: C1.+, C6.2, C8.2, C9.2, D5.C, IC2.4, J5.1, J6.1, PAD15.1, PAD16.1, PAD17.1, PAD18.1, PC2.+, R1.2, R3.2, R6.2, SL1.2, SL2.1, U$1.3, U$11.2, U$6.B1, U2.1, U2.3
- removed net +5V_3A: C27.+, IC1.4, U$10.2
- new net +5V_µC: C27.+, C6.2, D5.C, IC1.4, SL2.1, U$10.2, U$6.B1, U2.1, U2.3
- new net 22V: C16.+, C19.+, C20.+, C26.+, C30.+, C4.+, C5.+, IC2.1, LM2678S_ADJ.2, LM2678T-12.2, R8.1, U$6.K, X2.1
- new net BAT12_11V: J2.4, J3.1, R12.1
- new net BAT1_3.7V: J3.3, R14.1
- new net BAT1_7.4V: J3.2, R13.1
- new net BAT23_22V: J2.1, R9.1
- new net BAT2_14.8V: J2.3, R11.1
- new net BAT2_18.5V: J2.2, R10.1
- new net GND_POW: C1.-, C16.-, C18.-, C19.-, C20.-, C21.-, C23.2, C24.2, C25.2, C26.-, C28.-, C29.-, C30.-, C4.-, C5.-, IC2.3, IC2.5, J5.4, J6.4, LM2678S_ADJ.4, LM2678T-12.4, R15.2, U$2.A, U$3.A, U$5.A, X1.2, X10.2, X11.2, X15.2, X2.2, X3.2, X4.2, X9.2
- new net N$20: R13.2, U$13.P$1
- new net N$21: R10.2, U$13.P$14
- new net N$22: R14.2, U$13.P$5
- new net N$4: R9.2, U$13.P$15
- new net N$6: R11.2, U$13.P$13
- net +3V3: now also U$13.P$16
- net 5V_3A: now also C1.+, IC2.4, J5.1, J6.1, PAD15.1, PAD16.1, PAD17.1, PAD18.1, R1.2, R3.2, R6.2, U$1.3, U$11.2, X1.1; no longer X12.2
- net AN0/RA0: now also U$13.P$3; no longer PAD1.1
- net GND: now also ON1.C, R15.1, U$13.P$2, U$13.P$4, U$13.P$8; no longer C1.-, C16.-, C18.-, C19.-, C20.-, C21.-, C23.2, C24.2, C25.2, C26.-, C28.-, C29.-, C30.-, C4.-, C5.-, C8.1, C9.1, IC2.3, IC2.5, J1.4, J2.4, J5.4, J6.4, LM2678S_ADJ.4, LM2678T-12.4, PC2.-, SL1.1, U$2.A, U$3.A, U$5.A, X1.2, X10.2, X11.2, X12.1, X15.2, X9.2
- net N$15: now also R12.2, U$13.P$12; no longer C16.+, C19.+, C20.+, C26.+, C30.+, C4.+, C5.+, IC2.1, LM2678S_ADJ.2, LM2678T-12.2, R8.1, U$6.K, X1.1
- net N$17: now also X3.1
- net PWM1L2/RP13/RB13: now also R5.1
- net PWM2H1/RP22: now also U$13.P$9
- net PWM2L1/RP23/RC7: now also U$13.P$10
- net RA7: no longer ON1.C
- net RA8: no longer R5.1
- net RP24/RC8: now also U$13.P$11
- net RP25/RC9: now also U$13.P$6
- net V+: now also X4.1
Routing:
- net GND_POW: track 0.00 -> 533.5 mm
- net 22V: track 0.00 -> 270.9 mm, vias 0 -> 1
- net +5V_µC: track 0.00 -> 248.1 mm, vias 0 -> 2
- net 5V_3A: track 0.00 -> 201.4 mm, vias 0 -> 1
- net +3V3: track 0.00 -> 137.6 mm
- net N$17: track 0.00 -> 137.3 mm
- net V+: track 0.00 -> 119.2 mm
- net RA7: track 0.00 -> 109.5 mm, vias 0 -> 4
- net GND: track 0.00 -> 80.3 mm, vias 0 -> 23
- net RP21/RC5/RX/SS: track 0.00 -> 74.9 mm
- net RP20/TX/SDO: track 0.00 -> 71.6 mm
- net BAT3+: track 0.00 -> 71.4 mm
- net RESET: track 0.00 -> 54.9 mm
- net PGD: track 0.00 -> 51.8 mm
- net N$11: track 0.00 -> 49.4 mm
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- added copper zone on layer 1, net GND
- added copper zone on layer 16, net GND
