File: carte/alimentation/Alimv1.sch (EAGLE design)
At the start: 107 parts, among them IC1 LM2596T, IC2 LM2596T, IC4 DSPIC33FJ128MC804PT, J4 RJ11-2L-B, U2 LP2985-33DBVR, X10 22-23-2021, X11 22-23-2021, X9 22-23-2021

Commit message: alim v1
Reprise du travail des élèves
Parts:
- removed C8: 100n, SmartPrj:C-EU0603-RND
- removed C9: 100n, SmartPrj:C-EUC0603K
- removed J1: (no value), con-amp:MTA04-100
- removed LED1: RED, led:LED5MM
- removed PAD1: (no value), wirepad:1,6/0,9
- removed PC2: 47u, rcl:CPOL-EUD
- removed R16: 200, resistor:R-EU_R0805
- removed R17: 1600, resistor:R-EU_R0805
- removed R18: 1100, resistor:R-EU_R0805
- removed R19: 220, resistor:R-EU_R0805
- removed R20: 1300, resistor:R-EU_R0805
- removed SL1: (no value), con-amp-quick:M02
- removed X12: (no value), con-wago-500:W237-102
- added ON1: GREEN, led:LEDCHIP-LED0805
- added U$13: NX3L4051PW, Robot_MT:NX3L4051PW
- added X2, X3: MSTBV2, con-phoenix-508:MSTBV2
- added X4: 1751248, con-phoenix-350:1751248
- R10, R11: value 560 -> 20k; device resistor:R-EU_R0805 -> LibPerso:R-EU_R0805
- R12: value 300 -> 20k; device resistor:R-EU_R0805 -> LibPerso:R-EU_R0805
- R13: value 820 -> 20k; device resistor:R-EU_R0805 -> LibPerso:R-EU_R0805
- R14: value 240 -> 20k; device resistor:R-EU_R0805 -> LibPerso:R-EU_R0805
- R15: value 200 -> 0; device resistor:R-EU_R0805 -> LibPerso:R-EU_R0805
- R9: value 270 -> 20k; device resistor:R-EU_R0805 -> LibPerso:R-EU_R0805
- X1: value (none) -> MSTBV2; device con-wago-500:W237-102 -> con-phoenix-508:MSTBV2
Connections:
- removed net +5V: C1.+, C8.2, C9.2, IC2.FB, J5.1, J6.1, PAD15.P, PAD16.P, PAD17.P, PAD18.P, R1.2, R3.2, R6.2, SL2.1, U$1.VDD, U$11.2
- removed net +5V_3A: C27.+, C6.2, D5.C, IC1.FB, PC2.+, SL1.2, U$10.2, U$6G$1.1, U2.IN, U2.ON/!OFF
- removed net BAT3_25.9V: J1.3
- removed net BAT3_29.6V: J1.2
- removed net BAT3_33.3V: J1.1
- new net +5V_µC: C27.+, C6.2, D5.C, IC1.FB, SL2.1, U$10.2, U$6G$1.1, U2.IN, U2.ON/!OFF
- new net 22V: C16.+, C19.+, C20.+, C26.+, C30.+, C4.+, C5.+, IC2.VIN, LM2678S_ADJ.INPUT, LM2678T-12.INPUT, R8.1, U$6G$2.P, X2-1.1
- new net BAT12_11V: J2.4, J3.1, R12.1
- new net BAT23_22V: J2.1, R9.1
- new net GND_POW: C1.-, C16.-, C18.-, C19.-, C20.-, C21.-, C23.2, C24.2, C25.2, C26.-, C28.-, C29.-, C30.-, C4.-, C5.-, IC2.!ON!/OFF, IC2.GND, J5.4, J6.4, LM2678S_ADJ.GND, LM2678T-12.GND, R15.2, U$2.A, U$3.A, U$5.A, X1-2.1, X10-2.S, X11-2.S, X15-2.KL, X2-2.1, X3-2.1, X4-2.K, X9-2.S
- new net N$20: R13.2, U$13.Y4
- new net N$21: R10.2, U$13.Y1
- new net N$22: R14.2, U$13.Y5
- new net N$4: R9.2, U$13.Y2
- new net N$6: R11.2, U$13.Y0
- net +3V3: now also U$13.VCC
- net 5V_3A: now also C1.+, IC2.FB, J5.1, J6.1, PAD15.P, PAD16.P, PAD17.P, PAD18.P, R1.2, R3.2, R6.2, U$1.VDD, U$11.2, X1-1.1; no longer X12-2.KL
- net AN0/RA0: now also U$13.Z; no longer PAD1.P, R10.2, R9.2
- net AN1/RA1: no longer R11.2, R12.2
- net BAT12_11.1V: no longer J2.4, J3.1, R13.1
- net BAT1_3.7V: now also R14.1; no longer R9.1
- net BAT1_7.4V: now also R13.1; no longer R11.1
- net BAT23_22.2V: no longer J1.4, J2.1, R17.1
- net BAT2_14.8V: now also R11.1; no longer R18.1
- net BAT2_18.5V: now also R10.1; no longer R20.1
- net GND: now also ON1.C, U$13.GND, U$13.Y6, U$13.Y7; no longer C1.-, C16.-, C18.-, C19.-, C20.-, C21.-, C23.2, C24.2, C25.2, C26.-, C28.-, C29.-, C30.-, C4.-, C5.-, C8.1, C9.1, IC2.!ON!/OFF, IC2.GND, J5.4, J6.4, LM2678S_ADJ.GND, LM2678T-12.GND, PC2.-, R10.1, R12.1, R14.1, R16.1, R19.1, SL1.1, U$2.A, U$3.A, U$5.A, X1-2.KL, X10-2.S, X11-2.S, X12-1.KL, X15-2.KL, X9-2.S
- net N$1: now also ON1.A; no longer LED1.A
- net N$15: now also R12.2, U$13.Y3; no longer C16.+, C19.+, C20.+, C26.+, C30.+, C4.+, C5.+, IC2.VIN, LM2678S_ADJ.INPUT, LM2678T-12.INPUT, R8.1, U$6G$2.P, X1-1.KL
- net N$17: now also X3-1.1
- net PWM1L2/RP13/RB13: now also R5.1
- net PWM2H1/RP22: now also U$13.S3
- net PWM2L1/RP23/RC7: now also U$13.S2
- net RA7: no longer LED1.C
- net RA8: no longer R5.1
- net RP16/RC0/AN6: no longer R15.2, R20.2
- net RP17/RC1/AN7: no longer R16.2, R17.2
- net RP2/RB2/AN4: no longer R13.2, R14.2
- net RP24/RC8: now also U$13.S1
- net RP25/RC9: now also U$13.P$1
- net RP3/RB3/AN5: no longer R18.2, R19.2
- net V+: now also X4-1.K
Other:
- moved on the sheet: C1, C10, C11, C12, C13, C14, C15, C16, C17, C18, C19, C2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
